Commit message: move the arm and gripper for init

File: code/simulation/urdf/ur5_robotiq_85.urdf (robot description, URDF)
Before this commit: robot ur5_robotiq_85, 20 links, 19 joints
Joints:
- joint shoulder_lift_joint: type fixed -> revolute
- joint wrist_1_joint: type fixed -> revolute
- joint wrist_2_joint: type fixed -> revolute
- joint wrist_3_joint: type fixed -> revolute
