Commit message: make the box falling stable

File: code/simulation/urdf/blueBox.urdf (robot description, URDF)
Before this commit: robot cube, 1 links, 0 joints
Links:
- link right_leg: mass 20 -> 2000; geometry collision box size=0.1 0.3 0.1; visual box size=0.1 0.3 0.1

File: code/simulation/urdf/redBox.urdf (robot description, URDF)
Before this commit: robot cube, 1 links, 0 joints
Links:
- link right_leg: mass 20 -> 2000; geometry collision box size=0.1 0.3 0.1; visual box size=0.1 0.3 0.1
