Commit message: finish the env init

File: code/simulation/urdf/block.urdf (robot description, URDF)
Before this commit: robot conveyor_belt, 2 links, 1 joints
Links:
- link base_link: mass 10 -> 70; geometry collision box size=2 100 0.1; visual box size=2 100 0.1
- link belt_link: mass 10 -> 50; geometry collision box size=1 50 0.1; visual box size=1 50 0.1

File: code/simulation/urdf/blueBox.urdf (robot description, URDF)
Before this commit: robot cube, 1 links, 0 joints
Links:
- link right_leg: geometry collision box size=0.1 0.3 0.1; visual box size=0.1 0.3 0.1

File: code/simulation/urdf/greenBox.urdf (robot description, URDF)
Before this commit: robot cube, 1 links, 0 joints
Links:
- link right_leg: geometry collision box size=0.1 0.3 0.1; visual box size=0.1 0.3 0.1

File: code/simulation/urdf/redBox.urdf (robot description, URDF)
Before this commit: robot cube, 1 links, 0 joints
Links:
- link right_leg: geometry collision box size=0.1 0.3 0.1; visual box size=0.1 0.3 0.1

File: code/simulation/urdf/yellowBox.urdf (robot description, URDF)
Before this commit: robot conveyor_belt, 2 links, 1 joints
Links:
- removed link base_link
- removed link world
- added link right_leg, mass 1; collision box size=0.1 0.3 0.1; visual box size=0.1 0.3 0.1
Joints:
- removed joint joint_fix

Commit message: assign path to blocks

File: code/simulation/urdf/block.urdf (robot description, URDF)
Before this commit: robot conveyor_belt, 2 links, 1 joints
Links:
- link base_link: mass 70 -> 90; geometry collision box size=2 150 0.1; visual box size=2 150 0.1
- link belt_link: mass 50 -> 60; geometry collision box size=1 100 0.3; visual box size=1 100 0.3
Joints:
- joint prismatic_joint: limit lower=-500000000 upper=500000000 effort=500000000 velocity=5.0 -> lower=0 upper=500 effort=5000 velocity=5.0

File: code/simulation/urdf/blueBox.urdf (robot description, URDF)
Before this commit: robot cube, 1 links, 0 joints
Links:
- link right_leg: mass 1 -> 20

File: code/simulation/urdf/greenBox.urdf (robot description, URDF)
Before this commit: robot cube, 1 links, 0 joints
Links:
- link right_leg: mass 1 -> 20

File: code/simulation/urdf/redBox.urdf (robot description, URDF)
Before this commit: robot cube, 1 links, 0 joints
Links:
- link right_leg: mass 1 -> 20

Commit message: second time

File: code/simulation/urdf/block.urdf (robot description, URDF)
Before this commit: robot conveyor_belt, 2 links, 1 joints
Links:
- link base_link: geometry collision box size=5 150 0.1; visual box size=5 150 0.1
- link belt_link: geometry collision box size=0.7 100 0.3; visual box size=0.7 100 0.3

Commit message: try to train

File: code/simulation/urdf/block.urdf (robot description, URDF)
Before this commit: robot conveyor_belt, 2 links, 1 joints
Links:
- link base_link: geometry collision box size=10 150 0.1; visual box size=10 150 0.1
- link belt_link: geometry collision box size=.6 100 0.3; visual box size=.6 100 0.3

File: code/simulation/urdf/blueBox.urdf (robot description, URDF)
Before this commit: robot cube, 1 links, 0 joints
Links:
- link right_leg: geometry collision box size=0.1 0.2 0.1; visual box size=0.1 0.2 0.1

File: code/simulation/urdf/redBox.urdf (robot description, URDF)
Before this commit: robot cube, 1 links, 0 joints
Links:
- link right_leg: geometry collision box size=0.1 0.2 0.1; visual box size=0.1 0.2 0.1

Commit message: add green garbage, cube texture and remove gipper

File: code/simulation/urdf/block.urdf (robot description, URDF)
Before this commit: robot conveyor_belt, 2 links, 1 joints
Links:
- link belt_link: geometry collision box size=.6 100 0.15; visual box size=.6 100 0.15

File: code/simulation/urdf/blueBox.urdf (robot description, URDF)
Before this commit: robot cube, 1 links, 0 joints
Links:
- link right_leg: mass 2000 -> 200

File: code/simulation/urdf/redBox.urdf (robot description, URDF)
Before this commit: robot cube, 1 links, 0 joints
Links:
- link right_leg: mass 2000 -> 20

File: code/simulation/urdf/ur5_robotiq_85.urdf (robot description, URDF)
Before this commit: robot ur5_robotiq_85, 20 links, 19 joints
Links:
- link ee_link: geometry 
- link left_inner_finger: geometry visual mesh filename=../meshes/robotiq_85/visual/robotiq_arg2f_85_inner_finger.d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 scale=0.001 0.001 0.001
- link left_inner_finger_pad: geometry visual box size=0.022 0.00635 0.0375
- link left_inner_knuckle: geometry visual mesh filename=../meshes/robotiq_85/visual/robotiq_arg2f_85_inner_knuckle.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 scale=0.001 0.001 0.001
- link left_outer_finger: geometry visual mesh filename=../meshes/robotiq_85/visual/robotiq_arg2f_85_outer_finger.d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 scale=0.001 0.001 0.001
- link left_outer_knuckle: geometry visual mesh filename=../meshes/robotiq_85/visual/robotiq_arg2f_85_outer_knuckle.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 scale=0.001 0.001 0.001
- link right_inner_finger: geometry visual mesh filename=../meshes/robotiq_85/visual/robotiq_arg2f_85_inner_finger.d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 scale=0.001 0.001 0.001
- link right_inner_finger_pad: geometry visual box size=0.022 0.00635 0.0375
- link right_inner_knuckle: geometry visual mesh filename=../meshes/robotiq_85/visual/robotiq_arg2f_85_inner_knuckle.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 scale=0.001 0.001 0.001
- link right_outer_finger: geometry visual mesh filename=../meshes/robotiq_85/visual/robotiq_arg2f_85_outer_finger.d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 scale=0.001 0.001 0.001
- link right_outer_knuckle: geometry visual mesh filename=../meshes/robotiq_85/visual/robotiq_arg2f_85_outer_knuckle.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 scale=0.001 0.001 0.001
- link robotiq_arg2f_base_link: geometry visual mesh filename=../meshes/robotiq_85/visual/robotiq_arg2f_85_base_link.dae scale=0.001 0.001 0.001

Commit message: final

File: code/simulation/urdf/block.urdf (robot description, URDF)
Before this commit: robot conveyor_belt, 2 links, 1 joints
Links:
- link base_link: geometry collision box size=2 150 0.1; visual box size=2 150 0.1
- link belt_link: geometry collision box size=1 100 0.3; visual box size=1 100 0.3
